Commit message: make base_footprint parent

File: ws/src/cub_description/urdf/cub2023.xacro (robot description, xacro)
@@ -3,6 +3,5 @@
   <xacro:include filename="$(find cub_description)/urdf/cub2023_body.xacro" />
   <!-- <xacro:include filename="$(find cub_description)/urdf/cub2023_sensors.xacro" /> -->
-  <link name="base_link"/>
-  <xacro:cub_body parent="base_link"/>
+  <xacro:cub_body base_link="base_link" base_footprint="base_footprint"/>
   <!-- <xacro:cub_sensors parent="base_link"/> -->
 </robot>

File: ws/src/cub_description/urdf/cub2023_body.xacro (robot description, xacro)
@@ -1,17 +1,18 @@
 <?xml version="1.0"?>
 <robot name="cub2023_body" xmlns:xacro="http://ros.org/wiki/xacro">
-  <xacro:macro name="cub_body" params="parent">
+  <xacro:macro name="cub_body" params="base_link base_footprint">
     <material name="white">
       <color rgba="1.0 1.0 1.0 1.0"/>
     </material>
-    <link name="base_footprint"/>
+    <link name="${base_footprint}"/>
     <joint name="base_footprint_joint" type="fixed">
       <origin xyz="0.045 0 0" rpy="0 0 0" />
-      <parent link="${parent}" />
-      <child link="base_footprint" />
-    </joint>
+      <parent link="${base_footprint}" />
+      <child link="${base_link}" />
+    </joint>
+    <link name="${base_link}"/>
     <joint name="body_joint" type="fixed">
       <origin xyz="0 0 0" rpy="0 0 0" />
-      <parent link="${parent}" />
+      <parent link="${base_link}" />
       <child link="body" />
     </joint>
@@ -40,5 +41,5 @@
     <joint name="wheel_left_joint" type="continuous">
       <origin xyz="0.045 0.1225 0.1025" rpy="${-pi/2} 0 0" />
-      <parent link="${parent}" />
+      <parent link="${base_link}" />
       <child link="wheel_left" />
       <limit effort="1" velocity="1"/>
@@ -86,5 +87,5 @@
     <joint name="wheel_right_joint" type="continuous">
       <origin xyz="0.045 -0.1225 0.1025" rpy="${pi/2} 0 0" />
-      <parent link="${parent}" />
+      <parent link="${base_link}" />
       <child link="wheel_right" />
       <limit effort="1" velocity="1"/>
@@ -131,5 +132,5 @@
     <joint name="caster_joint" type="continuous">
       <origin xyz="-0.156 0.0 0.0" rpy="0 0 0" />
-      <parent link="${parent}" />
+      <parent link="${base_link}" />
       <child link="caster" />
       <limit effort="1" velocity="1"/>
@@ -160,5 +161,5 @@
     <joint name="head_joint" type="revolute">
       <origin xyz="-0.03989 0.0 0.66" rpy="0 0 0" />
-      <parent link="${parent}" />
+      <parent link="${base_link}" />
       <child link="head" />
       <limit effort="1" velocity="1" lower="0" upper="${pi/2}"/>
@@ -201,5 +202,5 @@
     <joint name="hokuyo_joint" type="fixed">
       <origin xyz="0.0 0.0 0.2342" rpy="0 0 0" />
-      <parent link="${parent}" />
+      <parent link="${base_link}" />
       <child link="hokuyo" />
     </joint>
@@ -218,5 +219,5 @@
     <joint name="hesai_joint" type="fixed">
       <origin xyz="-0.02 0.0 0.3947" rpy="0 0 0" />
-      <parent link="${parent}" />
+      <parent link="${base_link}" />
       <child link="hesai" />
     </joint>
