Commit message: robot_state_publisher.launch for real robot

File: ws/src/cub_description/urdf/cub2023_body.xacro (robot description, xacro)
@@ -45,4 +45,13 @@
       <axis xyz="0 0 1"/>
     </joint>
+    <transmission name="wheel_left_trans" type="SimpleTransmission">
+      <type>transmission_interface/SimpleTransmission</type>
+        <actuator name="wheel_left_motor">
+          <mechanicalReduction>1</mechanicalReduction>
+        </actuator>
+      <joint name="wheel_left_joint">
+        <hardwareInterface>hardware_interface/VelocityJointInterface</hardwareInterface>
+      </joint>
+    </transmission>
     <link name="wheel_left">
       <visual>
@@ -68,4 +77,11 @@
       </inertial>
     </link>
+    <gazebo reference="wheel_left">
+      <material>Gazebo/Black</material>
+      <mu1 value="10" />
+      <mu2 value="10" />
+      <kp value="10000" />
+      <kd value="100" />
+    </gazebo>
     <joint name="wheel_right_joint" type="continuous">
       <origin xyz="0.045 -0.1225 0.1025" rpy="${pi/2} 0 0" />
@@ -75,4 +91,13 @@
       <axis xyz="0 0 1"/>
     </joint>
+    <transmission name="wheel_right_trans" type="SimpleTransmission">
+      <type>transmission_interface/SimpleTransmission</type>
+        <actuator name="wheel_right_motor">
+          <mechanicalReduction>1</mechanicalReduction>
+        </actuator>
+      <joint name="wheel_right_joint">
+        <hardwareInterface>hardware_interface/VelocityJointInterface</hardwareInterface>
+      </joint>
+    </transmission>
     <link name="wheel_right">
       <visual>
@@ -97,4 +122,11 @@
       </inertial>
     </link>
+    <gazebo reference="wheel_right">
+      <material>Gazebo/Black</material>
+      <mu1 value="10" />
+      <mu2 value="10" />
+      <kp value="10000" />
+      <kd value="100" />
+    </gazebo>
     <joint name="caster_joint" type="continuous">
       <origin xyz="-0.156 0.0 0.0" rpy="0 0 0" />
@@ -133,4 +165,13 @@
       <axis xyz="0 1 0"/>
     </joint>
+    <transmission name="head_trans" type="SimpleTransmission">
+      <type>transmission_interface/SimpleTransmission</type>
+        <actuator name="head_motor">
+          <mechanicalReduction>1</mechanicalReduction>
+        </actuator>
+      <joint name="head_joint">
+        <hardwareInterface>hardware_interface/PositionJointInterface</hardwareInterface>
+      </joint>
+    </transmission>
     <link name="head">
       <visual>
@@ -155,4 +196,7 @@
       </inertial>
     </link>
+    <gazebo reference="head">
+      <material>Gazebo/White</material>
+    </gazebo>
     <joint name="hokuyo_joint" type="fixed">
       <origin xyz="0.0 0.0 0.2342" rpy="0 0 0" />
@@ -169,4 +213,7 @@
       </visual>
     </link>
+    <gazebo reference="hokuyo">
+      <material>Gazebo/Black</material>
+    </gazebo>
     <joint name="hesai_joint" type="fixed">
       <origin xyz="-0.02 0.0 0.3947" rpy="0 0 0" />
@@ -183,4 +230,14 @@
       </visual>
     </link>
+    <gazebo reference="hesai">
+      <material>Gazebo/White</material>
+    </gazebo>
+  <gazebo>
+    <plugin name="gazebo_ros_control" filename="libgazebo_ros_control.so">
+      <robotNamespace>/cub</robotNamespace>
+      <robotSimType>gazebo_ros_control/DefaultRobotHWSim</robotSimType>
+      <legacyModeNS>true</legacyModeNS>
+    </plugin>
+  </gazebo>
   </xacro:macro>
 </robot>

Commit message: update cub urdf for shibuya-san's

File: ws/src/cub_description/urdf/cub2023_body.xacro (robot description, xacro)
@@ -5,9 +5,17 @@
       <color rgba="1.0 1.0 1.0 1.0"/>
     </material>
-    <link name="${base_footprint}"/>
+    <!-- this is setting for "odometory -> base_footprint -> base_link" type  -->
+    <!-- <link name="${base_footprint}"/>
     <joint name="base_footprint_joint" type="fixed">
       <origin xyz="0.045 0 0" rpy="0 0 0" />
       <parent link="${base_footprint}" />
       <child link="${base_link}" />
+    </joint> -->
+    <!-- this is setting for "base_link -> odometory" type  -->
+    <link name="odometory"/>
+    <joint name="odometory_joint" type="fixed">
+      <origin xyz="0.045 0 0" rpy="0 0 0" />
+      <parent link="${base_link}" />
+      <child link="odometory" />
     </joint>
     <link name="${base_link}"/>
@@ -39,5 +47,5 @@
       </inertial>
     </link>
-    <joint name="wheel_left_joint" type="continuous">
+    <!-- <joint name="wheel_left_joint" type="continuous">
       <origin xyz="0.045 0.1225 0.1025" rpy="${-pi/2} 0 0" />
       <parent link="${base_link}" />
@@ -54,5 +62,10 @@
         <hardwareInterface>hardware_interface/VelocityJointInterface</hardwareInterface>
       </joint>
-    </transmission>
+    </transmission> -->
+    <joint name="wheel_left_joint" type="fixed">
+      <origin xyz="0.045 0.1225 0.1025" rpy="${-pi/2} 0 0" />
+      <parent link="${base_link}" />
+      <child link="wheel_left" />
+    </joint>
     <link name="wheel_left">
       <visual>
@@ -85,5 +98,5 @@
       <kd value="100" />
     </gazebo>
-    <joint name="wheel_right_joint" type="continuous">
+    <!-- <joint name="wheel_right_joint" type="continuous">
       <origin xyz="0.045 -0.1225 0.1025" rpy="${pi/2} 0 0" />
       <parent link="${base_link}" />
@@ -100,5 +113,10 @@
         <hardwareInterface>hardware_interface/VelocityJointInterface</hardwareInterface>
       </joint>
-    </transmission>
+    </transmission> -->
+    <joint name="wheel_right_joint" type="fixed">
+      <origin xyz="0.045 -0.1225 0.1025" rpy="${pi/2} 0 0" />
+      <parent link="${base_link}" />
+      <child link="wheel_right" />
+    </joint>
     <link name="wheel_right">
       <visual>
@@ -130,5 +148,5 @@
       <kd value="100" />
     </gazebo>
-    <joint name="caster_joint" type="continuous">
+    <!-- <joint name="caster_joint" type="continuous">
       <origin xyz="-0.156 0.0 0.0" rpy="0 0 0" />
       <parent link="${base_link}" />
@@ -136,5 +154,13 @@
       <limit effort="1" velocity="1"/>
       <axis xyz="0 0 1"/>
-    </joint>
+    </joint> -->
+    <joint name="caster_joint" type="fixed">
+      <origin xyz="-0.156 0.0 0.0" rpy="0 0 0" />
+      <parent link="${base_link}" />
+      <child link="caster" />
+    </joint>
+    <origin xyz="0.045 -0.1225 0.1025" rpy="${pi/2} 0 0" />
+      <parent link="${base_link}" />
+      <child link="wheel_right" />
     <link name="caster">
       <visual>
@@ -159,5 +185,5 @@
       </inertial>
     </link>
-    <joint name="head_joint" type="revolute">
+    <!-- <joint name="head_joint" type="revolute">
       <origin xyz="-0.03989 0.0 0.66" rpy="0 0 0" />
       <parent link="${base_link}" />
@@ -174,5 +200,10 @@
         <hardwareInterface>hardware_interface/PositionJointInterface</hardwareInterface>
       </joint>
-    </transmission>
+    </transmission> -->
+    <joint name="head_joint" type="fixed">
+      <origin xyz="-0.03989 0.0 0.66" rpy="0 ${30.0*pi/180.0} 0" />
+      <parent link="${base_link}" />
+      <child link="head" />
+    </joint>
     <link name="head">
       <visual>
@@ -217,10 +248,10 @@
       <material>Gazebo/Black</material>
     </gazebo>
-    <joint name="hesai_joint" type="fixed">
+    <joint name="Pandar_joint" type="fixed">
       <origin xyz="-0.02 0.0 0.3947" rpy="0 0 0" />
       <parent link="${base_link}" />
-      <child link="hesai" />
-    </joint>
-    <link name="hesai">
+      <child link="Pandar" />
+    </joint>
+    <link name="Pandar">
       <visual>
         <origin xyz="0 0 0" rpy="0 0 0"/>
@@ -231,5 +262,5 @@
       </visual>
     </link>
-    <gazebo reference="hesai">
+    <gazebo reference="Pandar">
       <material>Gazebo/White</material>
     </gazebo>

Commit message: honban

File: ws/src/cub_description/urdf/cub2023_body.xacro (robot description, xacro)
@@ -6,16 +6,16 @@
     </material>
     <!-- this is setting for "odometory -> base_footprint -> base_link" type  -->
-    <!-- <link name="${base_footprint}"/>
+    <link name="${base_footprint}"/>
     <joint name="base_footprint_joint" type="fixed">
       <origin xyz="0.045 0 0" rpy="0 0 0" />
       <parent link="${base_footprint}" />
       <child link="${base_link}" />
-    </joint> -->
-    <!-- this is setting for "base_link -> odometory" type  -->
-    <link name="odometory"/>
-    <joint name="odometory_joint" type="fixed">
+    </joint>
+    <!-- this is setting for "base_link -> odometry" type  -->
+    <link name="odometry"/>
+    <joint name="odometry_joint" type="fixed">
       <origin xyz="0.045 0 0" rpy="0 0 0" />
       <parent link="${base_link}" />
-      <child link="odometory" />
+      <child link="odometry" />
     </joint>
     <link name="${base_link}"/>
@@ -249,5 +249,5 @@
     </gazebo>
     <joint name="Pandar_joint" type="fixed">
-      <origin xyz="-0.02 0.0 0.3947" rpy="0 0 0" />
+      <origin xyz="-0.02 0.0 0.3947" rpy="0 0 ${90.0*pi/180.0}" />
       <parent link="${base_link}" />
       <child link="Pandar" />

Commit message: add imu launch and settings

File: ws/src/cub_description/urdf/cub2023_body.xacro (robot description, xacro)
@@ -265,4 +265,21 @@
       <material>Gazebo/White</material>
     </gazebo>
+    <joint name="imu_joint" type="fixed">
+      <origin xyz="-0.02 0.0 0.3" rpy="0 0 ${-90.0*pi/180.0}" />
+      <parent link="${base_link}" />
+      <child link="imu_link" />
+    </joint>
+    <link name="imu_link">
+      <visual>
+        <origin xyz="0 0 0" rpy="0 0 0"/>
+        <geometry>
+          <box size="0.05 0.05 0.02"/>
+        </geometry>
+        <material name="white"/>
+      </visual>
+    </link>
+    <gazebo reference="imu_link">
+      <material>Gazebo/White</material>
+    </gazebo>
   <gazebo>
     <plugin name="gazebo_ros_control" filename="libgazebo_ros_control.so">
