Commit message: add params file

File: ros/cub2_description/urdf/cub2.urdf (robot description, URDF)
Before this commit: robot cub2_robot, 8 links, 7 joints
Links:
- removed link velodyne_link
- added link velodyne; visual cylinder length=0.1 radius=0.05
Joints:
- joint base_to_footprint: child base_link -> base_footprint; parent base_footprint -> base_link
- joint base_to_velodyne: child velodyne_link -> velodyne
