Commit message: rename cub_description pkg definition

File: ros/cub_description/urdf/cub2.urdf (robot description, URDF)
Before this commit: robot cub2_robot, 8 links, 7 joints
Links:
- link base_link: geometry collision mesh filename=file://$(find cub_description)/meshes/Cub2URDF241001.dae scale=1 1 1; visual mesh filename=file://$(find cub_description)/meshes/Cub2URDF241001.dae scale=1 1 1

Commit message: add cub2 mesh

File: ros/cub_description/urdf/cub2.urdf (robot description, URDF)
Before this commit: robot cub2_robot, 8 links, 7 joints
Links:
- link base_link: geometry collision mesh filename=file://$(find cub_description)/meshes/cub2.dae scale=1 1 1; visual mesh filename=file://$(find cub_description)/meshes/cub2.dae scale=1 1 1
