Commit message: Update mesh file path resolution in URDF

File: ros/cub_description/urdf/spidar.urdf (robot description, URDF)
Before this commit: robot cub3_robot, 8 links, 7 joints
Links:
- link base_link: geometry collision mesh filename=package://cub_description/meshes/cub3.dae scale=1 1 1; visual mesh filename=package://cub_description/meshes/cub3.dae scale=1 1 1
