Commit message: Cub3

File: ros/cub_description/urdf/cub3.urdf (robot description, URDF)
Before this commit: robot cub2_robot, 8 links, 7 joints
Links:
- link base_link: geometry collision mesh filename=file://$(find cub_description)/meshes/cub3.dae scale=1 1 1; visual mesh filename=file://$(find cub_description)/meshes/cub3.dae scale=1 1 1

Commit message: adjust velodyne tilt

File: ros/cub_description/urdf/cub3.urdf (robot description, URDF)
Before this commit: robot cub3_robot, 8 links, 7 joints
Joints:
- joint base_to_velodyne: origin xyz=0.0 0 0.5 rpy=0 0 0 -> xyz=0.0 0 0.5 rpy=0 0.0361283 0

Commit message: update URDF

File: ros/cub_description/urdf/cub3.urdf (robot description, URDF)
Before this commit: robot cub3_robot, 8 links, 7 joints
Links:
- removed link SLCL_link
- removed link SLCR_link
- added link SLC1L; visual cylinder length=0.02 radius=0.03
- added link SLC1R; visual cylinder length=0.02 radius=0.03
Joints:
- joint base_to_SLCL: child SLCL_link -> SLC1L; origin xyz=-0.05 0.1 0.2 rpy=0 0 0 -> xyz=-0.05 0.1 0.2 rpy=0 0 -1.57079632679
- joint base_to_SLCR: child SLCR_link -> SLC1R; origin xyz=-0.05 -0.1 0.2 rpy=0 0 0 -> xyz=-0.05 -0.1 0.2 rpy=0 0 1.57079632679
- joint base_to_imu: origin xyz=0 0 0.1 rpy=0 0 0 -> xyz=0 0 0.48 rpy=0 0 0
