Commit message: rename codes cub3 to cub4

File: ros/cub_description/urdf/cub4.urdf (robot description, URDF)
Before this commit: robot cub3_robot, 8 links, 7 joints
Links:
- link base_link: geometry collision mesh filename=file://$(find cub_description)/meshes/cub4.dae scale=1 1 1; visual mesh filename=file://$(find cub_description)/meshes/cub4.dae scale=1 1 1

File: ros/cub_description/urdf/spidar.urdf (robot description, URDF)
Before this commit: robot cub3_robot, 8 links, 7 joints
Links:
- link base_link: geometry collision mesh filename=package://cub_description/meshes/cub4.dae scale=1 1 1; visual mesh filename=package://cub_description/meshes/cub4.dae scale=1 1 1

Commit message: update URDF

File: ros/cub_description/urdf/cub4.urdf (robot description, URDF)
Before this commit: robot cub4_robot, 8 links, 7 joints
Links:
- added link livox_frame; visual box size=0.015 0.015 0.015
Joints:
- added joint base_to_livox: type fixed, parent base_link, child livox_frame, origin xyz=0.0 0 0.6 rpy=0 0.785398 0
- joint base_to_velodyne: origin xyz=0.0 0 0.5 rpy=0 0.0361283 0 -> xyz=0.0 0 0.3 rpy=0 0.0361283 0

Commit message: update sensor pose

File: ros/cub_description/urdf/cub4.urdf (robot description, URDF)
Before this commit: robot cub4_robot, 9 links, 8 joints
Links:
- removed link SLC1L
- removed link SLC1R
- removed link gps_link
- added link gnss_main_link
- added link gnss_sub_link
- link base_footprint: geometry 
- link base_link: geometry collision mesh filename=file://$(find cub_description)/meshes/cub4-comp.obj scale=0.1 0.1 0.1; visual mesh filename=file://$(find cub_description)/meshes/cub4-comp.obj scale=0.1 0.1 0.1
- link camera_link: geometry 
- link imu_link: geometry 
- link livox_frame: geometry 
- link velodyne: geometry 
Joints:
- removed joint base_to_SLCL
- removed joint base_to_SLCR
- removed joint base_to_gps
- added joint base_to_gnss_main: type fixed, parent base_link, child gnss_main_link, origin xyz=-0.12 0.1 0.5857 rpy=0 0 0
- added joint base_to_gnss_sub: type fixed, parent base_link, child gnss_sub_link, origin xyz=-0.12 -0.1 0.5857 rpy=0 0 0
- joint base_to_camera: origin xyz=0.0 0 0.4 rpy=0 0 0 -> xyz=-0.0589 0 0.5020 rpy=0 0.1745 0
- joint base_to_imu: origin xyz=0 0 0.48 rpy=0 0 0 -> xyz=-0.030 0 0.2034 rpy=3.14 0 0
- joint base_to_livox: origin xyz=0.0 0 0.6 rpy=0 0.785398 0 -> xyz=-0.0379 0 0.5779 rpy=0 0.7854 0
- joint base_to_velodyne: origin xyz=0.0 0 0.3 rpy=0 0.0361283 0 -> xyz=0.0 0 0.2492 rpy=0 0 0

Commit message: bugfix for geometry

File: ros/cub_description/urdf/cub4.urdf (robot description, URDF)
Before this commit: robot cub4_robot, 8 links, 7 joints
Links:
- removed link camera_link
- added link oak_parent_frame
Joints:
- joint base_to_camera: child camera_link -> oak_parent_frame
