Commit message: fix for new env

File: ros/mcub_bringup/urdf/mcub.urdf.xacro (robot description, xacro)
@@ -1,4 +1,5 @@
 <?xml version="1.0"?>
-<robot name="mcub" xmlns:xacro="http://www.ros.org/wiki/xacro">
+<robot name="mcub" xmlns:xacro="http://www.ros.org/wiki/xacro"
+       xmlns:cubsim="https://github.com/tomoki-na/Cub_ROS/cubsim">
   <!--
     mCub simulation model template.
@@ -30,5 +31,5 @@
   <xacro:arg name="base_cog_x" default="-0.045"/>
   <xacro:arg name="base_cog_y" default="0.000"/>
-  <xacro:arg name="base_cog_z" default="0.070"/>
+  <xacro:arg name="base_cog_z" default="0.040"/>
   <xacro:arg name="base_ixx" default="0.0020"/>
   <xacro:arg name="base_ixy" default="0.0"/>
@@ -39,5 +40,5 @@
   <!-- Wheel diameter is confirmed. Track requires resolving the 0.130/0.125 m discrepancy above. -->
   <xacro:arg name="wheel_radius" default="0.020"/>
-  <xacro:arg name="wheel_track" default="0.130"/>
+  <xacro:arg name="wheel_track" default="0.125"/>
   <xacro:arg name="wheel_x" default="0.000"/>
   <xacro:arg name="wheel_width" default="0.015"/>
@@ -66,6 +67,4 @@
   <xacro:arg name="caster_wheel_iyy" default="0.000004"/>
   <xacro:arg name="caster_wheel_izz" default="0.000005"/>
-  <xacro:arg name="caster_swivel_damping" default="0.02"/>
-  <xacro:arg name="caster_axle_damping" default="0.005"/>
   <!--
     The LiDAR visual geometry follows cub_description/urdf/mcub.urdf:
@@ -132,6 +131,4 @@
   <xacro:property name="caster_wheel_iyy" value="$(arg caster_wheel_iyy)"/>
   <xacro:property name="caster_wheel_izz" value="$(arg caster_wheel_izz)"/>
-  <xacro:property name="caster_swivel_damping" value="$(arg caster_swivel_damping)"/>
-  <xacro:property name="caster_axle_damping" value="$(arg caster_axle_damping)"/>
   <xacro:property name="lidar_scan_x" value="$(arg lidar_scan_x)"/>
   <xacro:property name="lidar_scan_y" value="$(arg lidar_scan_y)"/>
@@ -217,12 +214,13 @@
   <xacro:drive_wheel side="left" y="${wheel_track / 2}" sign="1"/>
   <xacro:drive_wheel side="right" y="${-wheel_track / 2}" sign="1"/>
-  <!-- Passive trailing caster: free swivel about z plus free wheel rotation about y. -->
-  <joint name="caster_swivel_joint" type="continuous">
+  <!--
+    Stable simulation approximation: preserve the caster frames and visual wheel,
+    but use fixed joints and a spherical contact shape. This behaves as a ball
+    caster without an undamped swivel degree of freedom or faceted wheel contact.
+  -->
+  <joint name="caster_swivel_joint" type="fixed">
     <parent link="base_link"/>
     <child link="caster_swivel_link"/>
     <origin xyz="${caster_pivot_x} 0 ${caster_pivot_z}" rpy="0 0 0"/>
-    <axis xyz="0 0 1"/>
-    <limit effort="0.1" velocity="30.0"/>
-    <dynamics damping="${caster_swivel_damping}" friction="0.0"/>
   </joint>
   <link name="caster_swivel_link">
@@ -247,11 +245,8 @@
     </collision>
   </link>
-  <joint name="caster_wheel_joint" type="continuous">
+  <joint name="caster_wheel_joint" type="fixed">
     <parent link="caster_swivel_link"/>
     <child link="caster_wheel_link"/>
     <origin xyz="${-caster_trail} 0 ${caster_wheel_radius - caster_pivot_z}" rpy="0 0 0"/>
-    <axis xyz="0 1 0"/>
-    <limit effort="0.1" velocity="30.0"/>
-    <dynamics damping="${caster_axle_damping}" friction="0.0"/>
   </joint>
   <link name="caster_wheel_link">
@@ -269,7 +264,6 @@
     </visual>
     <collision>
-      <origin rpy="${pi / 2} 0 0"/>
-      <geometry>
-        <cylinder radius="${caster_wheel_radius}" length="${caster_wheel_width}"/>
+      <geometry>
+        <sphere radius="${caster_wheel_radius}"/>
       </geometry>
     </collision>
@@ -323,3 +317,6 @@
     </collision>
   </link>
+  <!-- CubSim Editor import metadata. UnitySensorsROS is intentionally not used. -->
+  <cubsim:sensor name="slc1" type="raycast_lidar" link="SLC1_link"
+                 frequency="10.0" samples="500" min_range="0.05" max_range="12.0"/>
 </robot>

File: unity/CubSim/Assets/Cub/Generated/Import/mcub.urdf (robot description, URDF)
Before this commit: robot mcub, 8 links, 7 joints
Links:
- link caster_wheel_link: geometry collision cylinder length=0.012 radius=0.02; visual cylinder length=0.012 radius=0.02
Joints:
- joint caster_swivel_joint: axis (none) -> 0 0 1; limit (none) -> effort=0.1 velocity=30.0; type fixed -> continuous
- joint caster_wheel_joint: axis (none) -> 0 1 0; limit (none) -> effort=0.1 velocity=30.0; type fixed -> continuous
